File: PSA-Harness/kicad_project/PSA-Harness.kicad_sch (KiCad schematic)
At the start: 20 parts, among them J1 to_EPS_1, J10 B2B_1, J11 B2B_2, J2 to_EPS_2, J3 to_ESP_3, J4 to_car_1, J5 to_car_2, J6 to_car_3, J7 USB_C_Receptacle, J8 B2B_1, J9 B2B_2, U1 DG419LEUA, U2 DG419LEUA

Commit message: cable-board setup
Parts:
- removed J10, J8: B2B_1, Connector_PinHeader_1.27mm:PinHeader_2x15_P1.27mm_Vertical, symbol Connector_Generic:Conn_02x15_Odd_Even
- removed J11, J9: B2B_2, Connector_PinHeader_1.27mm:PinHeader_2x15_P1.27mm_Vertical, symbol Connector_Generic:Conn_02x15_Odd_Even
- J4, J5, J6: footprint PSA:ESW-110-44-F-D -> PSA:10129381-920003BLF
- J7: footprint PSA:GCT_USB4115-03-C_REVB4 -> PSA:TYPE-C-31-M-04
Other:
- note added: "Harness Connector"
- note added: "OBD-C Connector"
- note added: "Solid State Relay"
- note added: "Voltage Protection"
- note removed: "Harness Connector (PCB1)"
- note removed: "Harness Connector (PCB2)"
- note removed: "OBD-C Connector (PCB2)"
- note removed: "Solid State Relay (PCB2)"
- note removed: "Voltage Protection (PCB2)"
- moved on the sheet: J1, J2, J3, J4, J5, J6

Commit message: move to_car connector to back side
Parts:
- J4, J5, J6: footprint PSA:10129381-920003BLF -> PSA:10129381-920003BLF_BACK
Changed lines of the file:
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@@
 			)
 		)
-		(property "Footprint" "PSA:10129381-920003BLF"
+		(property "Footprint" "PSA:10129381-920003BLF_BACK"
 			(at 109.22 82.55 0)
 			(effects
@@
 			)
 		)
-		(property "Footprint" "PSA:10129381-920003BLF"
+		(property "Footprint" "PSA:10129381-920003BLF_BACK"
 			(at 78.74 82.55 0)
 			(effects
@@
 			)
 		)
-		(property "Footprint" "PSA:10129381-920003BLF"
+		(property "Footprint" "PSA:10129381-920003BLF_BACK"
 			(at 48.26 82.55 0)
 			(effects

Commit message: use other USB-C connector
Parts:
- J7: footprint PSA:TYPE-C-31-M-04 -> PSA:GCT_USB4056-03-A_REVA2
Changed lines of the file:
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@@
 			)
 		)
-		(property "Footprint" "PSA:TYPE-C-31-M-04"
+		(property "Footprint" "PSA:GCT_USB4056-03-A_REVA2"
 			(at 247.65 69.85 0)
 			(effects
