File: PSA-Harness/kicad_project/PCB2.kicad_pcb (KiCad board)
At the start: 4 copper layers, 28.3 x 54 mm, 15 parts, among them J1 to_EPS_1, J2 to_EPS_2, J3 to_ESP_3, J7 USB_C_Receptacle, J8 B2B_1, J9 B2B_2, U1 DG419LEUA, U2 DG419LEUA

Commit message: change footprint of analog switch from msop to soic on pcb2
Parts:
- U1, U2: footprint Package_SO:MSOP-8_3x3mm_P0.65mm -> Package_SO:SOIC-8_3.9x4.9mm_P1.27mm
- moved D3 0.66 mm to (97.9, 95.3)
- moved U1 0.60 mm to (97.9, 95.4)
Routing:
- net CAN0_L: track 55.2 -> 0.00 mm, vias 2 -> 0
- net +12V: track 81.0 -> 40.9 mm, vias 1 -> 0
- net SBU1: track 32.7 -> 0.00 mm, vias 1 -> 0
- net CAN0_H: track 61.3 -> 32.2 mm, vias 2 -> 0
- net CAN2_H: track 23.3 -> 12.7 mm, vias 3 -> 1
- net CAN2_L: track 38.8 -> 28.5 mm
- net Net-(R2-Pad1): track 7.85 -> 0.00 mm, vias 2 -> 0
- net Net-(R1-Pad2): track 4.77 -> 0.00 mm
- net GND: vias 52 -> 33

Commit message: PCB2 routed
Parts:
- moved D2 5.20 mm to (108.7, 95.3)
- moved D1 5.00 mm to (113.7, 95.3)
Routing:
- net CAN0_L: track 0.00 -> 62.6 mm, vias 0 -> 2
- net +12V: track 40.9 -> 81.5 mm, vias 0 -> 4
- net SBU1: track 0.00 -> 37.2 mm, vias 0 -> 1
- net CAN0_H: track 32.2 -> 61.8 mm, vias 0 -> 2
- net CAN2_H: track 12.7 -> 24.9 mm, vias 1 -> 2
- net CAN2_L: track 28.5 -> 38.0 mm, vias 0 -> 2
- net Net-(R2-Pad1): track 0.00 -> 7.65 mm, vias 0 -> 2
- net Net-(R1-Pad2): track 0.00 -> 4.72 mm
- net GND: vias 33 -> 52

Commit message: PCB2 add up indicator
Other:
- board text added: "up"
Changed lines of the file:
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@@
+		(layer "F.SilkS")
+	)
+	(gr_line
+		(start 108.4 106.125)
+		(end 107.6 107)
+		(stroke
+			(width 0.2)
+			(type solid)
+		)
+		(layer "F.SilkS")
+	)
+	(gr_line
+		(start 109.2 107)
+		(end 108.4 106.125)
+		(stroke
+			(width 0.2)
+			(type solid)
+		)
 		(layer "F.SilkS")
 	)
@@
 		)
 		(fill yes)
+		(layer "F.SilkS")
+	)
+	(gr_line
+		(start 108.4 108.2)
+		(end 108.4 106.125)
+		(stroke
+			(width 0.2)
+			(type solid)
+		)
 		(layer "F.SilkS")
 	)
@@
 		(layer "Edge.Cuts")
 	)
+	(gr_text "up"
+		(at 103.2 108 0)
+		(layer "F.SilkS")
+		(effects
+			(font
+				(size 2 2)
+				(thickness 0.25)
+			)
+			(justify left bottom)
+		)
+	)
 	(gr_text "PCB1"
