File: PSA-Harness/kicad_tester/PSA-Tester/PSA-Tester.kicad_sch (KiCad schematic)
At the start: 8 parts, among them U1 MCP23017_SO, U2 MCP23017_SO, U3 MCP23017_SO, U4 MCP23017_SO, U5 MCP23017_SO, U6 MCP23017_SO, U7 MCP23017_SO, U8 MCP23017_SO

Commit message: initial tester schematic done
Parts:
- added C1, C2, C3: 100n, symbol Device:C
- added J1, J10, J2, J3, J4, J5, J6, J7, J8, J9: ~, symbol Connector_Generic:Conn_02x10_Counter_Clockwise
- added J11: USB_C_Receptacle, symbol Connector:USB_C_Receptacle
- added R1, R2, R3, R4, R5, R6, R7, R8: 10k, symbol Device:R
- added SW1, SW2, SW3: SW_Push, symbol Switch:SW_Push
- added U10: ESP32-C3-OLED, symbol 0_tester:ESP32-C3-OLED
- added U9: MCP23017_SO, Package_SO:SOIC-28W_7.5x17.9mm_P1.27mm, symbol Interface_Expansion:MCP23017_SO
Connections:
- net +3V3: now also R1.1, R2.1, R3.1, R4.1, R5.1, SW1.1, SW2.1, SW3.1, U10. (3), U9.9 (VDD)
- net GND: now also C1.2, C2.2, C3.2, R6.2, R7.2, R8.2, U10. (3), U9.10 (VSS), U9.15 (A0), U9.16 (A1), U9.17 (A2)
- net 33: now reaches U3.1 (GPB0)
- net 33: now also J2.18 (Pin_18), J5.18 (Pin_18)
- net nRESET: now reaches U3.18 (~{RESET})
- net nRESET: now also U1.18 (~{RESET}), U2.18 (~{RESET}), U4.18 (~{RESET}), U5.18 (~{RESET}), U6.18 (~{RESET}), U7.18 (~{RESET}), U8.18 (~{RESET}), R1.2, U10. (3), U9.18 (~{RESET})
- net 34: now reaches U3.2 (GPB1)
- net 34: now also J2.17 (Pin_17), J5.17 (Pin_17)
- net 41: now reaches U3.21 (GPA0)
- net 41: now also J3.1 (Pin_1)
- net 42: now reaches U3.22 (GPA1)
- net 42: now also J3.2 (Pin_2)
- net 43: now reaches U3.23 (GPA2)
- net 43: now also J3.3 (Pin_3)
- net 44: now reaches U3.24 (GPA3)
- net 44: now also J3.4 (Pin_4)
- net 45: now reaches U3.25 (GPA4)
- net 45: now also J3.5 (Pin_5)
- net 46: now reaches U3.26 (GPA5)
- net 46: now also J3.6 (Pin_6)
- net 47: now reaches U3.27 (GPA6)
- net 47: now also J3.7 (Pin_7)
- net 48: now reaches U3.28 (GPA7)
- net 48: now also J3.8 (Pin_8)
- net 35: now reaches U3.3 (GPB2)
- net 35: now also J2.16 (Pin_16), J5.16 (Pin_16)
- net 36: now reaches U3.4 (GPB3)
- net 36: now also J2.15 (Pin_15), J5.15 (Pin_15)
- net 37: now reaches U3.5 (GPB4)
- net 37: now also J2.14 (Pin_14), J5.14 (Pin_14)
- net 38: now reaches U3.6 (GPB5)
- net 38: now also J2.13 (Pin_13), J5.13 (Pin_13)
- net 39: now reaches U3.7 (GPB6)
- net 39: now also J2.12 (Pin_12), J5.12 (Pin_12)
- net 40: now reaches U3.8 (GPB7)
- net 40: now also J2.11 (Pin_11), J5.11 (Pin_11)
- net 49a: now reaches U8.1 (GPB0)
- net 49a: now also J10.9 (Pin_9)
- net 50a: now reaches U8.2 (GPB1)
- net 50a: now also J10.10 (Pin_10)
- net 57a: now reaches U8.21 (GPA0)
- net 57a: now also J10.14 (Pin_14)
- net 58a: now reaches U8.22 (GPA1)
- net 58a: now also J10.13 (Pin_13)
- net 59a: now reaches U8.23 (GPA2)
- net 59a: now also J10.12 (Pin_12)
- net 60a: now reaches U8.24 (GPA3)
- net 60a: now also J10.11 (Pin_11)
- net 61: now reaches U8.25 (GPA4)
- net 61: now also J11.A4 (VBUS), J11.A9 (VBUS), J11.B4 (VBUS), J11.B9 (VBUS)
- net 62: now reaches U8.26 (GPA5)
- net 62: now also J11.A5 (CC1)
- net 63: now reaches U8.27 (GPA6)
- net 63: now also J11.B5 (CC2)
- net 64: now reaches U8.28 (GPA7)
- net 64: now also J11.A7 (D-)
- net 51a: now reaches U8.3 (GPB2)
- net 51a: now also J10.20 (Pin_20)
- net 52a: now reaches U8.4 (GPB3)
- net 52a: now also J10.19 (Pin_19)
- net 53a: now reaches U8.5 (GPB4)
- net 53a: now also J10.18 (Pin_18)
- net 54a: now reaches U8.6 (GPB5)
- net 54a: now also J10.17 (Pin_17)
- net 55a: now reaches U8.7 (GPB6)
- net 55a: now also J10.16 (Pin_16)
- net 56a: now reaches U8.8 (GPB7)
- net 56a: now also J10.15 (Pin_15)
- net 49: now reaches U4.1 (GPB0)
- net 49: now also J3.9 (Pin_9)
- net 50: now reaches U4.2 (GPB1)
- net 50: now also J3.10 (Pin_10)
- net 57: now reaches U4.21 (GPA0)
- net 57: now also J3.14 (Pin_14)
- net 58: now reaches U4.22 (GPA1)
- net 58: now also J3.13 (Pin_13)
- net 59: now reaches U4.23 (GPA2)
- net 59: now also J3.12 (Pin_12)
- net 60: now reaches U4.24 (GPA3)
- net 60: now also J3.11 (Pin_11)
- net 51: now reaches U4.3 (GPB2)
- net 51: now also J3.20 (Pin_20)
- net 52: now reaches U4.4 (GPB3)
- net 52: now also J3.19 (Pin_19)
- net 53: now reaches U4.5 (GPB4)
- net 53: now also J3.18 (Pin_18)
- net 54: now reaches U4.6 (GPB5)
- net 54: now also J3.17 (Pin_17)
- net 55: now reaches U4.7 (GPB6)
- net 55: now also J3.16 (Pin_16)
- net 56: now reaches U4.8 (GPB7)
- net 56: now also J3.15 (Pin_15)
- net 33a: now reaches U7.1 (GPB0)
- net 33a: now also J8.18 (Pin_18), J9.18 (Pin_18)
- net 34a: now reaches U7.2 (GPB1)
- net 34a: now also J8.17 (Pin_17), J9.17 (Pin_17)
- net 41a: now reaches U7.21 (GPA0)
- net 41a: now also J10.1 (Pin_1)
- net 42a: now reaches U7.22 (GPA1)
- net 42a: now also J10.2 (Pin_2)
- net 43a: now reaches U7.23 (GPA2)
- net 43a: now also J10.3 (Pin_3)
- net 44a: now reaches U7.24 (GPA3)
- net 44a: now also J10.4 (Pin_4)
- net 45a: now reaches U7.25 (GPA4)
- net 45a: now also J10.5 (Pin_5)
- net 46a: now reaches U7.26 (GPA5)
- net 46a: now also J10.6 (Pin_6)
- net 47a: now reaches U7.27 (GPA6)
- net 47a: now also J10.7 (Pin_7)
- net 48a: now reaches U7.28 (GPA7)
- net 48a: now also J10.8 (Pin_8)
- net 35a: now reaches U7.3 (GPB2)
- net 35a: now also J8.16 (Pin_16), J9.16 (Pin_16)
- net 36a: now reaches U7.4 (GPB3)
- net 36a: now also J8.15 (Pin_15), J9.15 (Pin_15)
- net 37a: now reaches U7.5 (GPB4)
- net 37a: now also J8.14 (Pin_14), J9.14 (Pin_14)
- net 38a: now reaches U7.6 (GPB5)
- net 38a: now also J8.13 (Pin_13), J9.13 (Pin_13)
- net 39a: now reaches U7.7 (GPB6)
- net 39a: now also J8.12 (Pin_12), J9.12 (Pin_12)
- net 40a: now reaches U7.8 (GPB7)
- net 40a: now also J8.11 (Pin_11), J9.11 (Pin_11)
- net 17a: now reaches U6.1 (GPB0)
- net 17a: now also J6.14 (Pin_14), J7.14 (Pin_14)
- net 18a: now reaches U6.2 (GPB1)
- net 18a: now also J6.13 (Pin_13), J7.13 (Pin_13)
- net 25a: now reaches U6.21 (GPA0)
- net 25a: now also J8.5 (Pin_5), J9.5 (Pin_5)
- net 26a: now reaches U6.22 (GPA1)
- net 26a: now also J8.6 (Pin_6), J9.6 (Pin_6)
- net 27a: now reaches U6.23 (GPA2)
- net 27a: now also J8.7 (Pin_7), J9.7 (Pin_7)
- net 28a: now reaches U6.24 (GPA3)
- net 28a: now also J8.8 (Pin_8), J9.8 (Pin_8)
- net 29a: now reaches U6.25 (GPA4)
- net 29a: now also J8.9 (Pin_9), J9.9 (Pin_9)
- net 30a: now reaches U6.26 (GPA5)
- net 30a: now also J8.10 (Pin_10), J9.10 (Pin_10)
- net 31a: now reaches U6.27 (GPA6)
- net 31a: now also J8.20 (Pin_20), J9.20 (Pin_20)
- net 32a: now reaches U6.28 (GPA7)
- net 32a: now also J8.19 (Pin_19), J9.19 (Pin_19)
- net 19a: now reaches U6.3 (GPB2)
- net 19a: now also J6.12 (Pin_12), J7.12 (Pin_12)
- net 20a: now reaches U6.4 (GPB3)
- net 20a: now also J6.11 (Pin_11), J7.11 (Pin_11)
- net 21a: now reaches U6.5 (GPB4)
- net 21a: now also J8.1 (Pin_1), J9.1 (Pin_1)
- net 22a: now reaches U6.6 (GPB5)
- net 22a: now also J8.2 (Pin_2), J9.2 (Pin_2)
- net 23a: now reaches U6.7 (GPB6)
- net 23a: now also J8.3 (Pin_3), J9.3 (Pin_3)
- net 24a: now reaches U6.8 (GPB7)
- net 24a: now also J8.4 (Pin_4), J9.4 (Pin_4)
- net 1: now reaches U1.1 (GPB0)
- net 1: now also J1.1 (Pin_1), J4.1 (Pin_1)
- net 2: now reaches U1.2 (GPB1)
- net 2: now also J1.2 (Pin_2), J4.2 (Pin_2)
- net 9: now reaches U1.21 (GPA0)
- net 9: now also J1.9 (Pin_9), J4.9 (Pin_9)
- net 10: now reaches U1.22 (GPA1)
- net 10: now also J1.10 (Pin_10), J4.10 (Pin_10)
- net 11: now reaches U1.23 (GPA2)
- net 11: now also J1.20 (Pin_20), J4.20 (Pin_20)
- net 12: now reaches U1.24 (GPA3)
- net 12: now also J1.19 (Pin_19), J4.19 (Pin_19)
- net 13: now reaches U1.25 (GPA4)
- net 13: now also J1.18 (Pin_18), J4.18 (Pin_18)
- net 14: now reaches U1.26 (GPA5)
- net 14: now also J1.17 (Pin_17), J4.17 (Pin_17)
- net 15: now reaches U1.27 (GPA6)
- net 15: now also J1.16 (Pin_16), J4.16 (Pin_16)
- net 16: now reaches U1.28 (GPA7)
- net 16: now also J1.15 (Pin_15), J4.15 (Pin_15)
- net 3: now reaches U1.3 (GPB2)
- net 3: now also J1.3 (Pin_3), J4.3 (Pin_3)
- net 4: now reaches U1.4 (GPB3)
- net 4: now also J1.4 (Pin_4), J4.4 (Pin_4)
- net 5: now reaches U1.5 (GPB4)
- net 5: now also J1.5 (Pin_5), J4.5 (Pin_5)
- net 6: now reaches U1.6 (GPB5)
- net 6: now also J1.6 (Pin_6), J4.6 (Pin_6)
- net 7: now reaches U1.7 (GPB6)
- net 7: now also J1.7 (Pin_7), J4.7 (Pin_7)
- net 8: now reaches U1.8 (GPB7)
- net 8: now also J1.8 (Pin_8), J4.8 (Pin_8)
- net 1a: now reaches U5.1 (GPB0)
- net 1a: now also J6.1 (Pin_1), J7.1 (Pin_1)
- net 2a: now reaches U5.2 (GPB1)
- net 2a: now also J6.2 (Pin_2), J7.2 (Pin_2)
- net 9a: now reaches U5.21 (GPA0)
- net 9a: now also J6.9 (Pin_9), J7.9 (Pin_9)
- net 10a: now reaches U5.22 (GPA1)
- net 10a: now also J6.10 (Pin_10), J7.10 (Pin_10)
- net 11a: now reaches U5.23 (GPA2)
- net 11a: now also J6.20 (Pin_20), J7.20 (Pin_20)
- net 12a: now reaches U5.24 (GPA3)
- net 12a: now also J6.19 (Pin_19), J7.19 (Pin_19)
- net 13a: now reaches U5.25 (GPA4)
- net 13a: now also J6.18 (Pin_18), J7.18 (Pin_18)
- net 14a: now reaches U5.26 (GPA5)
- net 14a: now also J6.17 (Pin_17), J7.17 (Pin_17)
- net 15a: now reaches U5.27 (GPA6)
- net 15a: now also J6.16 (Pin_16), J7.16 (Pin_16)
- net 16a: now reaches U5.28 (GPA7)
- net 16a: now also J6.15 (Pin_15), J7.15 (Pin_15)
- net 3a: now reaches U5.3 (GPB2)
- net 3a: now also J6.3 (Pin_3), J7.3 (Pin_3)
- net 4a: now reaches U5.4 (GPB3)
- net 4a: now also J6.4 (Pin_4), J7.4 (Pin_4)
- net 5a: now reaches U5.5 (GPB4)
- net 5a: now also J6.5 (Pin_5), J7.5 (Pin_5)
- net 6a: now reaches U5.6 (GPB5)
- net 6a: now also J6.6 (Pin_6), J7.6 (Pin_6)
- net 7a: now reaches U5.7 (GPB6)
- net 7a: now also J6.7 (Pin_7), J7.7 (Pin_7)
- net 8a: now reaches U5.8 (GPB7)
- net 8a: now also J6.8 (Pin_8), J7.8 (Pin_8)
- net 17: now reaches U2.1 (GPB0)
- net 17: now also J1.14 (Pin_14), J4.14 (Pin_14)
- net 18: now reaches U2.2 (GPB1)
- net 18: now also J1.13 (Pin_13), J4.13 (Pin_13)
- net 25: now reaches U2.21 (GPA0)
- net 25: now also J2.5 (Pin_5), J5.5 (Pin_5)
- net 26: now reaches U2.22 (GPA1)
- net 26: now also J2.6 (Pin_6), J5.6 (Pin_6)
- net 27: now reaches U2.23 (GPA2)
- net 27: now also J2.7 (Pin_7), J5.7 (Pin_7)
- net 28: now reaches U2.24 (GPA3)
- net 28: now also J2.8 (Pin_8), J5.8 (Pin_8)
- net 29: now reaches U2.25 (GPA4)
- net 29: now also J2.9 (Pin_9), J5.9 (Pin_9)
- net 30: now reaches U2.26 (GPA5)
- net 30: now also J2.10 (Pin_10), J5.10 (Pin_10)
- net 31: now reaches U2.27 (GPA6)
- net 31: now also J2.20 (Pin_20), J5.20 (Pin_20)
- net 32: now reaches U2.28 (GPA7)
- net 32: now also J2.19 (Pin_19), J5.19 (Pin_19)
- net 19: now reaches U2.3 (GPB2)
- net 19: now also J1.12 (Pin_12), J4.12 (Pin_12)
- net 20: now reaches U2.4 (GPB3)
- net 20: now also J1.11 (Pin_11), J4.11 (Pin_11)
- net 21: now reaches U2.5 (GPB4)
- net 21: now also J2.1 (Pin_1), J5.1 (Pin_1)
- net 22: now reaches U2.6 (GPB5)
- net 22: now also J2.2 (Pin_2), J5.2 (Pin_2)
- net 23: now reaches U2.7 (GPB6)
- net 23: now also J2.3 (Pin_3), J5.3 (Pin_3)
- net 24: now reaches U2.8 (GPB7)
- net 24: now also J2.4 (Pin_4), J5.4 (Pin_4)
- net SCL renamed SCL1
- net SCL1: now also R5.2, U10. (3)
- net SDA renamed SDA1
- net SDA1: now also R4.2, U10. (3)
- new net 65: J11.B7 (D-), U9.1 (GPB0)
- new net 66: J11.A6 (D+), U9.2 (GPB1)
- new net 67: J11.B6 (D+), U9.3 (GPB2)
- new net 68: J11.B10 (RX1-), U9.4 (GPB3)
- new net 69: J11.B11 (RX1+), U9.5 (GPB4)
- new net 70: J11.A3 (TX1-), U9.6 (GPB5)
- new net 71: J11.A2 (TX1+), U9.7 (GPB6)
- new net 72: J11.A10 (RX2-), U9.8 (GPB7)
- new net 73: J11.A11 (RX2+), U9.21 (GPA0)
- new net 74: J11.B3 (TX2-), U9.22 (GPA1)
- new net 75: J11.B2 (TX2+), U9.23 (GPA2)
- new net 76: J11.A8 (SBU1), U9.24 (GPA3)
- new net 77: J11.B8 (SBU2), U9.25 (GPA4)
- new net 78: J11.A1 (GND), J11.A12 (GND), J11.B1 (GND), J11.B12 (GND), U9.26 (GPA5)
- new net 79: J11.S1 (SHIELD), U9.27 (GPA6)
- new net BUTTON1: C1.1, R6.1, SW1.2, U10. (3)
- new net BUTTON2: C2.1, R7.1, SW2.2, U10. (3)
- new net BUTTON3: C3.1, R8.1, SW3.2, U10. (3)
- new net SCL2: R3.2, U10. (3), U9.12 (SCK)
- new net SDA2: R2.2, U10. (3), U9.13 (SDA)
- no-connect marks 0 -> 29
Other:
- note added: "Controller"
- note added: "MEB Plug"
- note added: "MEB Socket"
- note added: "Multiplexer"
- note added: "OBC-C"
- note added: "PSA Plug"
- note added: "PSA Socket"
- moved on the sheet: U1, U2, U3, U4, U5, U6, U7, U8
