File: PSA-Harness/kicad_tester/PSA-Tester/PSA-Tester.kicad_pcb (KiCad board)
At the start: 4 copper layers, 100 x 100 mm, 41 parts, among them J11 U262-241N-4BV60, M1 MountingHole_3.2mm_M3_Pad_Via, M2 MountingHole_3.2mm_M3_Pad_Via, M3 MountingHole_3.2mm_M3_Pad_Via, M4 MountingHole_3.2mm_M3_Pad_Via, SW1 B3S-1000, SW2 B3S-1000, SW3 B3S-1000, U1 MCP23017T-E/SO, U10 ESP32-C3-OLED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

Commit message: routed
Parts:
- D1: value WS2812C-2020-V1 -> XL-0807RGBC-WS2812B
Routing:
- net 8: track 0.00 -> 117.3 mm, vias 0 -> 3
- net nRESET: track 112.6 -> 217.0 mm, vias 0 -> 3
- net 9: track 0.00 -> 99.8 mm, vias 0 -> 2
- net 40: track 0.00 -> 97.3 mm, vias 0 -> 2
- net 4: track 0.00 -> 93.5 mm, vias 0 -> 2
- net 26: track 0.00 -> 93.1 mm, vias 0 -> 2
- net 38: track 0.00 -> 87.9 mm, vias 0 -> 2
- net 17: track 0.00 -> 85.2 mm, vias 0 -> 2
- net 6: track 0.00 -> 83.7 mm, vias 0 -> 2
- net 24: track 0.00 -> 82.4 mm, vias 0 -> 3
- net 22: track 0.00 -> 81.5 mm, vias 0 -> 1
- net 21: track 0.00 -> 78.5 mm, vias 0 -> 2
- net 25: track 0.00 -> 78.0 mm, vias 0 -> 1
- net 2: track 0.00 -> 78.0 mm, vias 0 -> 1
- net 31a: track 0.00 -> 77.0 mm, vias 0 -> 1
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
Commit message: fixes
Parts:
- moved C4 0.80 mm to (105.7, 49.1)
Routing:
- net +3V3: track 62.0 -> 65.2 mm, vias 32 -> 31
- net 42: track 49.7 -> 48.1 mm

Commit message: usb-c footprint fix
Routing:
- net 6: track 83.7 -> 82.2 mm
- net 55: track 32.2 -> 32.9 mm
- net GND: vias 66 -> 58
Changed lines of the file:
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@@
 		(pad "S1" thru_hole oval
 			(at -4.49 1.4)
-			(size 0.95 1.8)
-			(drill oval 0.5 1.2)
+			(size 1 1.8)
+			(drill oval 0.62 1.2)
 			(layers "*.Cu" "*.Mask")
 			(remove_unused_layers no)
@@
 		(pad "S1" thru_hole oval
 			(at -4.13 -3.11)
-			(size 0.8 1.4)
-			(drill oval 0.5 1.1)
+			(size 0.9 1.4)
+			(drill oval 0.62 1.1)
 			(layers "*.Cu" "*.Mask")
 			(remove_unused_layers no)
@@
 		(pad "S1" thru_hole oval
 			(at 4.13 -3.11)
-			(size 0.8 1.4)
-			(drill oval 0.5 1.1)
+			(size 0.9 1.4)
+			(drill oval 0.62 1.1)
 			(layers "*.Cu" "*.Mask")
 			(remove_unused_layers no)
@@
 		(pad "S1" thru_hole oval
 			(at 4.49 1.4)
-			(size 0.95 1.8)
-			(drill oval 0.5 1.2)
+			(size 1 1.8)
+			(drill oval 0.62 1.2)
 			(layers "*.Cu" "*.Mask")
 			(remove_unused_layers no)
@@
 	)
 	(gr_text "plug"
-		(at 80 65 0)
+		(at 80.07 64.95 0)
 		(layer "F.SilkS")
 		(effects
@@
 	)
 	(gr_text "plug"
-		(at 42 65 0)
+		(at 42 64.86 0)
 		(layer "F.SilkS")
 		(effects
@@
 	)
 	(via
-		(at 137 51.5)
-		(size 0.5)
-		(drill 0.3)
-		(layers "F.Cu" "B.Cu")
-		(free yes)
-		(net 1)
-	)
-	(via
 		(at 44.2 83)
 		(size 0.5)
@@
 	)
 	(via
-		(at 40.5 51.5)
-		(size 0.5)
-		(drill 0.3)
-		(layers "F.Cu" "B.Cu")
-		(free yes)
-		(net 1)
-	)
-	(via
 		(at 71.6 102.95)
 		(size 0.5)
@@
 	)
 	(via
-		(at 47.5 44.5)
-		(size 0.5)
-		(drill 0.3)
-		(layers "F.Cu" "B.Cu")
-		(free yes)
-		(net 1)
-	)
-	(via
 		(at 86 52)
 		(size 0.5)
@@
 	)
 	(via
-		(at 41 135)
-		(size 0.5)
-		(drill 0.3)
-		(layers "F.Cu" "B.Cu")
-		(free yes)
-		(net 1)
-	)
-	(via
 		(at 90.9 83.05)
 		(size 0.5)
@@
 	)
 	(via
-		(at 131 44.5)
-		(size 0.5)
-		(drill 0.3)
-		(layers "F.Cu" "B.Cu")
-		(free yes)
-		(net 1)
-	)
-	(via
 		(at 111 94.5)
 		(size 0.5)
@@
 	)
 	(via
-		(at 85 63)
+		(at 85.33 62.996866)
 		(size 0.5)
 		(drill 0.3)
@@
 	)
 	(via
-		(at 136.5 134)
-		(size 0.5)
-		(drill 0.3)
-		(layers "F.Cu" "B.Cu")
-		(free yes)
-		(net 1)
-	)
-	(via
 		(at 95.5 47.5)
 		(size 0.5)
@@
 	)
 	(via
-		(at 47.5 141.5)
-		(size 0.5)
-		(drill 0.3)
-		(layers "F.Cu" "B.Cu")
-		(free yes)
-		(net 1)
-	)
-	(via
 		(at 81.1 85)
 		(size 0.5)
@@
 	)
 	(via
-		(at 130.5 140.5)
-		(size 0.5)
-		(drill 0.3)
-		(layers "F.Cu" "B.Cu")
-		(free yes)
-		(net 1)
-	)
-	(via
 		(at 97 94.5)
 		(size 0.5)
@@
 	)
 	(via
-		(at 42.566 51.35)
+		(at 43.31 51.58)
 		(size 0.5)
 		(drill 0.3)
@@
 	)
 	(segment
-		(start 42.566 51.35)
-		(end 42.566 75.845)
+		(start 40.177 54.713)
+		(end 43.31 51.58)
 		(width 0.2)
 		(layer "In1.Cu")
@@
 	)
 	(segment
-		(start 42.566 75.845)
-		(end 40.177 78.234)
+		(start 40.177 78.234)
+		(end 40.177 54.713)
 		(width 0.2)
 		(layer "In1.Cu")
@@
 	)
 	(segment
-		(start 42.566 51.35)
-		(end 44.9976 48.9184)
-		(width 0.2)
-		(layer "In2.Cu")
-		(net 18)
-	)
-	(segment
 		(start 72.5147 50.1807)
 		(end 71.4944 51.201)
@@
 	)
 	(segment
-		(start 53.0384 48.9184)
-		(end 54.2 50.08)
+		(start 54.2 50.08)
+		(end 52.93 51.35)
+		(width 0.2)
+		(layer "In2.Cu")
+		(net 18)
+	)
+	(segment
+		(start 52.93 51.35)
+		(end 43.54 51.35)
 		(width 0.2)
 		(layer "In2.Cu")
@@
 	)
 	(segment
-		(start 73.9589 51.201)
-		(end 72.9386 50.1807)
+		(start 43.54 51.35)
+		(end 43.31 51.58)
 		(width 0.2)
 		(layer "In2.Cu")
@@
 	)
 	(segment
-		(start 55.321 51.201)
-		(end 54.2 50.08)
+		(start 73.9589 51.201)
+		(end 72.9386 50.1807)
 		(width 0.2)
 		(layer "In2.Cu")
@@
 	)
 	(segment
-		(start 44.9976 48.9184)
-		(end 53.0384 48.9184)
+		(start 55.321 51.201)
+		(end 54.2 50.08)
 		(width 0.2)
 		(layer "In2.Cu")
@@
 	)
 	(via
-		(at 84.114 64.3941)
+		(at 84.11 63.15)
 		(size 0.5)
 		(drill 0.3)
@@
 	)
 	(segment
-		(start 84.114 76.2157)
-		(end 86.2735 78.3752)
+		(start 84.11 76.2117)
+		(end 84.11 63.15)
 		(width 0.2)
 		(layer "In1.Cu")
@@
 	)
 	(segment
-		(start 84.114 64.3941)
-		(end 84.114 76.2157)
+		(start 86.2735 78.3752)
+		(end 84.11 76.2117)
 		(width 0.2)
 		(layer "In1.Cu")
@@
 	)
 	(segment
-		(start 82.4999 62.78)
-		(end 84.114 64.3941)
+		(start 83.74 62.78)
+		(end 84.11 63.15)
 		(width 0.2)
 		(layer "In2.Cu")
@@
 	(segment
 		(start 71 62.78)
-		(end 82.4999 62.78)
+		(end 83.74 62.78)
 		(width 0.2)
 		(layer "In2.Cu")
@@
 	)
 	(segment
-		(start 112.1505 136.7872)
-		(end 112.1505 101.3825)
+		(start 115.09 136.86)
+		(end 114.15 137.8)
 		(width 0.2)
 		(layer "In1.Cu")
@@
 	)
 	(segment
-		(start 115.09 136.86)
-		(end 114.2112 137.7388)
+		(start 112.94 137.8)
+		(end 112.1505 137.0105)
 		(width 0.2)
 		(layer "In1.Cu")
@@
 	)
 	(segment
-		(start 114.2112 137.7388)
-		(end 113.1021 137.7388)
+		(start 114.15 137.8)
+		(end 112.94 137.8)
 		(width 0.2)
 		(layer "In1.Cu")
@@
 	)
 	(segment
-		(start 113.1021 137.7388)
-		(end 112.1505 136.7872)
+		(start 112.1505 137.0105)
+		(end 112.1505 101.3825)
 		(width 0.2)
 		(layer "In1.Cu")
@@
 	)
 	(segment
-		(start 107.2538 132.2092)
-		(end 107.2538 96.4985)
+		(start 107.6875 133.1575)
+		(end 107.6875 132.6429)
 		(width 0.2)
 		(layer "In1.Cu")
@@
 	)
 	(segment
-		(start 115.89 136.86)
-		(end 115.89 136.9634)
+		(start 115.89 137.319619)
+		(end 115.049619 138.16)
 		(width 0.2)
 		(layer "In1.Cu")
@@
 	)
 	(segment
-		(start 115.89 136.9634)
-		(end 114.7287 138.1247)
+		(start 107.6875 132.6429)
+		(end 107.2538 132.2092)
 		(width 0.2)
 		(layer "In1.Cu")
@@
 	)
 	(segment
-		(start 107.6875 132.6429)
-		(end 107.2538 132.2092)
+		(start 107.2538 96.4985)
+		(end 106.5921 95.8368)
 		(width 0.2)
 		(layer "In1.Cu")
@@
 	)
 	(segment
-		(start 112.9488 138.1247)
-		(end 107.6875 132.8634)
+		(start 112.69 138.16)
+		(end 107.6875 133.1575)
 		(width 0.2)
 		(layer "In1.Cu")
@@
 	)
 	(segment
-		(start 107.2538 96.4985)
-		(end 106.5921 95.8368)
+		(start 115.89 136.86)
+		(end 115.89 137.319619)
 		(width 0.2)
 		(layer "In1.Cu")
@@
 	)
 	(segment
-		(start 107.6875 132.8634)
-		(end 107.6875 132.6429)
+		(start 107.2538 132.2092)
+		(end 107.2538 96.4985)
 		(width 0.2)
 		(layer "In1.Cu")
@@
 	)
 	(segment
-		(start 114.7287 138.1247)
-		(end 112.9488 138.1247)
+		(start 115.049619 138.16)
+		(end 112.69 138.16)
 		(width 0.2)
 		(layer "In1.Cu")
