File: PSA-MEB-Harness-Tester/kicad_project/PSA-Tester.kicad_pcb (KiCad board)
At the start: 4 copper layers, 100 x 100 mm, 41 parts, among them J11 TYPE-C-31-M-04, SW1 TS-1057S-03126, SW2 TS-1057S-03126, SW3 TS-1057S-03126, U1 MCP23017T-E/SO, U10 ESP32-C3-OLED, U2 MCP23017T-E/SO, U3 MCP23017T-E/SO, U4 MCP23017T-E/SO, U5 MCP23017T-E/SO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

Commit message: fix DRC
Routing:
- net 1: track 73.9 -> 81.9 mm
Changed lines of the file:
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@@
 	)
 	(via
-		(at 91.446 43.3491)
+		(at 95.63 44.15)
 		(size 0.5)
 		(drill 0.3)
@@
 	)
 	(segment
-		(start 89.96 45)
-		(end 89.96 43.8883)
+		(start 43.6612 70.5103)
+		(end 43.6612 53.8326)
 		(width 0.2)
 		(layer "In1.Cu")
@@
 	)
 	(segment
-		(start 43.6612 70.5103)
-		(end 43.6612 53.8326)
+		(start 91.4 43.56)
+		(end 95.04 43.56)
 		(width 0.2)
 		(layer "In1.Cu")
@@
 	)
 	(segment
-		(start 90.9068 43.8883)
-		(end 91.446 43.3491)
+		(start 89.96 45)
+		(end 91.4 43.56)
 		(width 0.2)
 		(layer "In1.Cu")
@@
 	)
 	(segment
-		(start 89.96 43.8883)
-		(end 90.9068 43.8883)
+		(start 95.04 43.56)
+		(end 95.63 44.15)
 		(width 0.2)
 		(layer "In1.Cu")
@@
 	)
 	(segment
-		(start 54.1447 43.3491)
-		(end 52.7717 44.7221)
-		(width 0.2)
-		(layer "In2.Cu")
-		(net 17)
-	)
-	(segment
-		(start 52.7717 44.7221)
-		(end 52.7717 45)
+		(start 51.66 45)
+		(end 53.3109 43.3491)
 		(width 0.2)
 		(layer "In2.Cu")
@@
 	)
 	(segment
-		(start 91.446 43.3491)
-		(end 54.1447 43.3491)
+		(start 53.3109 43.3491)
+		(end 94.8291 43.3491)
 		(width 0.2)
 		(layer "In2.Cu")
@@
 	)
 	(segment
-		(start 51.66 45)
-		(end 52.7717 45)
+		(start 94.8291 43.3491)
+		(end 95.63 44.15)
 		(width 0.2)
 		(layer "In2.Cu")
@@
 	)
 	(via
-		(at 91.2516 71.7709)
+		(at 91.25 72.28)
 		(size 0.5)
 		(drill 0.3)
@@
 	)
 	(segment
-		(start 92.5 65.32)
+		(start 91.2516 72.2784)
 		(end 91.2516 66.5684)
 		(width 0.2)
@@
 	)
 	(segment
+		(start 91.25 72.28)
+		(end 91.2516 72.2784)
+		(width 0.2)
+		(layer "B.Cu")
+		(net 23)
+	)
+	(segment
 		(start 91.2516 66.5684)
-		(end 91.2516 71.7709)
+		(end 92.5 65.32)
 		(width 0.2)
 		(layer "B.Cu")
@@
 	)
 	(segment
-		(start 89.4264 73.5961)
-		(end 56.9817 73.5961)
+		(start 56.9817 73.5961)
+		(end 56.7037 73.8741)
 		(width 0.2)
 		(layer "In2.Cu")
@@
 	)
 	(segment
-		(start 91.2516 71.7709)
+		(start 90.7425 72.28)
 		(end 89.4264 73.5961)
 		(width 0.2)
@@
 	)
 	(segment
-		(start 56.9817 73.5961)
-		(end 56.7037 73.8741)
+		(start 91.25 72.28)
+		(end 90.7425 72.28)
+		(width 0.2)
+		(layer "In2.Cu")
+		(net 23)
+	)
+	(segment
+		(start 89.4264 73.5961)
+		(end 56.9817 73.5961)
 		(width 0.2)
 		(layer "In2.Cu")
@@
 	(segment
 		(start 98.36 45)
-		(end 97.2483 45)
+		(end 95.61 45)
 		(width 0.2)
 		(layer "F.Cu")
@@
 	)
 	(segment
-		(start 58.3 76.735)
-		(end 58.9659 76.0691)
+		(start 94.4983 43.8883)
+		(end 62.0054 43.8883)
 		(width 0.2)
 		(layer "F.Cu")
@@
 	)
 	(segment
-		(start 60.06 45)
-		(end 61.1717 45)
+		(start 58.3 76.735)
+		(end 58.9659 76.0691)
 		(width 0.2)
 		(layer "F.Cu")
@@
 	)
 	(segment
-		(start 58.9659 76.0691)
-		(end 60.0499 76.0691)
+		(start 61.1717 45)
+		(end 60.06 45)
 		(width 0.2)
 		(layer "F.Cu")
@@
 	)
 	(segment
-		(start 97.2483 45)
-		(end 96.1366 43.8883)
+		(start 58.9659 76.0691)
+		(end 60.0499 76.0691)
 		(width 0.2)
 		(layer "F.Cu")
@@
 	)
 	(segment
-		(start 96.1366 43.8883)
-		(end 62.0054 43.8883)
+		(start 95.61 45)
+		(end 94.4983 43.8883)
 		(width 0.2)
 		(layer "F.Cu")
@@
 	)
 	(segment
-		(start 85.0736 100.6955)
+		(start 81.884018 99.8427)
 		(end 84.2208 99.8427)
 		(width 0.2)
@@
 	)
 	(segment
-		(start 81.8337 99.8427)
-		(end 81.6329 100.0435)
+		(start 89.1495 100.6955)
+		(end 89.4 100.445)
 		(width 0.2)
 		(layer "F.Cu")
@@
 	)
 	(segment
-		(start 89.1495 100.6955)
+		(start 84.2208 99.8427)
 		(end 85.0736 100.6955)
 		(width 0.2)
@@
 	)
 	(segment
-		(start 89.4 100.445)
+		(start 85.0736 100.6955)
 		(end 89.1495 100.6955)
 		(width 0.2)
@@
 		(net 106)
 	)
-	(segment
-		(start 84.2208 99.8427)
-		(end 81.8337 99.8427)
-		(width 0.2)
-		(layer "F.Cu")
-		(net 106)
-	)
 	(via
-		(at 81.6329 100.0435)
+		(at 81.884018 99.8427)
 		(size 0.5)
 		(drill 0.3)
@@
 	)
 	(segment
-		(start 75.04 127.7)
+		(start 81.6329 100.093818)
+		(end 81.6329 100.5078)
+		(width 0.2)
+		(layer "In1.Cu")
+		(net 106)
+	)
+	(segment
+		(start 81.2883 100.8524)
 		(end 81.2883 121.4517)
 		(width 0.2)
@@
 	)
 	(segment
-		(start 81.6329 100.5078)
-		(end 81.6329 100.0435)
+		(start 81.884018 99.8427)
+		(end 81.6329 100.093818)
 		(width 0.2)
 		(layer "In1.Cu")
@@
 	)
 	(segment
-		(start 81.2883 121.4517)
+		(start 81.6329 100.5078)
 		(end 81.2883 100.8524)
 		(width 0.2)
@@
 	)
 	(segment
-		(start 81.2883 100.8524)
-		(end 81.6329 100.5078)
+		(start 81.2883 121.4517)
+		(end 75.04 127.7)
 		(width 0.2)
 		(layer "In1.Cu")
@@
 	)
 	(segment
-		(start 118.33 98.5607)
-		(end 118.33 94.6966)
+		(start 124.33 136.16)
+		(end 124.26 136.09)
 		(width 0.2)
 		(layer "In1.Cu")
@@
 	)
 	(segment
-		(start 124.33 136.16)
-		(end 124.33 132.3126)
+		(start 124.63 132.28)
+		(end 124.63 131.5)
 		(width 0.2)
 		(layer "In1.Cu")
@@
 	)
 	(segment
-		(start 124.33 131.6456)
-		(end 124.33 104.5607)
+		(start 124.26 136.09)
+		(end 124.26 132.65)
 		(width 0.2)
 		(layer "In1.Cu")
@@
 	)
 	(segment
-		(start 124.4515 132.1911)
-		(end 124.4515 131.7671)
+		(start 124.33 131.2)
+		(end 124.33 104.5607)
 		(width 0.2)
 		(layer "In1.Cu")
@@
 	)
 	(segment
-		(start 124.4515 131.7671)
-		(end 124.33 131.6456)
+		(start 118.33 98.5607)
+		(end 118.33 94.6966)
 		(width 0.2)
 		(layer "In1.Cu")
@@
 	)
 	(segment
-		(start 124.33 132.3126)
-		(end 124.4515 132.1911)
+		(start 124.63 131.5)
+		(end 124.33 131.2)
 		(width 0.2)
 		(layer "In1.Cu")
@@
 	)
 	(segment
+		(start 124.26 132.65)
+		(end 124.63 132.28)
+		(width 0.2)
+		(layer "In1.Cu")
+		(net 131)
+	)
+	(segment
 		(start 107.7542 96.64)
 		(end 109.2375 98.1233)
@@
 	)
 	(segment
-		(start 125.8688 105.5864)
-		(end 121.2954 101.013)
+		(start 121.2954 101.013)
+		(end 121.2954 96.8554)
 		(width 0.2)
 		(layer "In1.Cu")
@@
 	)
 	(segment
-		(start 121.2954 101.013)
-		(end 121.2954 96.8554)
+		(start 126.04 136.38)
+		(end 126.04 105.7576)
 		(width 0.2)
 		(layer "In1.Cu")
@@
 	)
 	(segment
-		(start 125.66 136.76)
-		(end 125.8688 136.5512)
+		(start 117.3703 92.9303)
+		(end 116.4043 92.9303)
 		(width 0.2)
 		(layer "In1.Cu")
@@
 	)
 	(segment
-		(start 121.2954 96.8554)
-		(end 117.3703 92.9303)
+		(start 126.04 105.7576)
+		(end 121.2954 101.013)
 		(width 0.2)
 		(layer "In1.Cu")
@@
 	)
 	(segment
-		(start 117.3703 92.9303)
-		(end 116.4043 92.9303)
+		(start 125.66 136.76)
+		(end 126.04 136.38)
 		(width 0.2)
 		(layer "In1.Cu")
@@
 	)
 	(segment
-		(start 125.8688 136.5512)
-		(end 125.8688 105.5864)
+		(start 121.2954 96.8554)
+		(end 117.3703 92.9303)
 		(width 0.2)
 		(layer "In1.Cu")
@@
 	)
 	(segment
-		(start 126.6849 137.4824)
-		(end 126.6849 101.2529)
+		(start 126.77 137.3973)
+		(end 126.77 101.647984)
+		(width 0.2)
+		(layer "In1.Cu")
+		(net 140)
+	)
+	(segment
+		(start 126.77 101.647984)
+		(end 126.75 101.627983)
 		(width 0.2)
 		(layer "In1.Cu")
@@
 	)
 	(segment
-		(start 126.6849 101.2529)
+		(start 126.75 101.627983)
+		(end 126.75 101.318)
+		(width 0.2)
+		(layer "In1.Cu")
+		(net 140)
+	)
+	(segment
+		(start 126.75 101.318)
 		(end 120.774 95.342)
 		(width 0.2)
@@
 	(segment
 		(start 126.0839 138.0834)
-		(end 126.6849 137.4824)
+		(end 126.77 137.3973)
 		(width 0.2)
 		(layer "In1.Cu")
@@
 	)
 	(segment
-		(start 123.93 136.86)
-		(end 124.7917 137.7217)
+		(start 126.41 137.2458)
+		(end 126.41 101.7971)
 		(width 0.2)
 		(layer "In1.Cu")
@@
 	)
 	(segment
-		(start 126.3232 137.3326)
-		(end 126.3232 101.7103)
+		(start 126.41 101.7971)
+		(end 122.2219 97.609)
 		(width 0.2)
 		(layer "In1.Cu")
@@
 	)
 	(segment
-		(start 124.7917 137.7217)
-		(end 125.9341 137.7217)
+		(start 123.93 136.86)
+		(end 124.7917 137.7217)
 		(width 0.2)
 		(layer "In1.Cu")
@@
 	)
 	(segment
-		(start 126.3232 101.7103)
-		(end 122.2219 97.609)
+		(start 125.9341 137.7217)
+		(end 126.41 137.2458)
 		(width 0.2)
 		(layer "In1.Cu")
@@
 	)
 	(segment
-		(start 125.9341 137.7217)
-		(end 126.3232 137.3326)
+		(start 124.7917 137.7217)
+		(end 125.9341 137.7217)
 		(width 0.2)
 		(layer "In1.Cu")
